File: hard/v2.0/chordboard/chordboard.kicad_pcb (KiCad board)
At the start: 2 copper layers, 302.9 x 193 mm, 278 parts, among them J1 T_UART0, J2 E_I2C0, J3 E_UART0, J4 T_UART5, J5 T_I2C0, J6 ++5V_IN, J7 Conn_01x07, SW1 SW_Push, SW10 SW_Push, SW11 SW_Push, SW12 SW_Push, SW13 SW_Push, SW14 SW_Push, SW15 SW_Push, SW16 SW_Push, SW17 SW_Push, SW18 SW_Push, SW19 SW_Push, SW2 SW_Push, SW20 SW_Push, SW21 SW_Push, SW22 SW_Push, SW23 SW_Push, SW24 SW_Push, SW25 SW_Push, SW26 SW_Push, SW27 SW_Push, SW28 SW_Push, SW29 SW_Push, SW3 SW_Push, SW30 SW_Push, SW31 SW_Push, SW32 SW_Push, SW33 SW_Push, SW34 SW_Push, SW35 SW_Push, SW36 SW_Push, SW37 SW_Push, SW38 SW_Push, SW39 SW_Push, SW4 SW_Push, SW40 SW_Push, SW41 SW_Push, SW42 SW_Push, SW43 SW_Push, SW44 SW_Push, SW45 SW_Push, SW46 SW_Push, SW47 SW_Push, SW48 SW_Push, SW5 SW_Push, SW6 SW_Push, SW7 SW_Push, SW8 SW_Push, SW9 SW_Push, U1 ESP32-WROVER, U2 AZ1117-3.3, U3 74LS126, U4 MCP73832-2-OT

Commit message: Updated
Parts:
- removed C1 (x2), C17, C18, C2 (x2), C22, C23: C, Capacitor_THT:C_Disc_D3.0mm_W1.6mm_P2.50mm
- removed the C11 at (469.4, -84.0)
- removed C19, C20, C21, C5 (x3), C6 (x4): C_Small, Capacitor_THT:C_Disc_D3.0mm_W2.0mm_P2.50mm
- removed C3 (x2): 10uF, Capacitor_THT:CP_Radial_D5.0mm_P2.00mm
- removed C4 (x2): 100uF, Capacitor_THT:CP_Radial_D5.0mm_P2.00mm
- removed D1, D2: D, Diode_THT:D_DO-41_SOD81_P7.62mm_Horizontal
- removed H1, H2, H5, H6: MountingHole, MountingHole:MountingHole_2.7mm_M2.5_Pad_Via
- removed HT1, HT2: HT16K33, Package_SO:SOIC-28W_7.5x17.9mm_P1.27mm
- removed JP3: J_ESP_RST, Jumper:SolderJumper-2_P1.3mm_Bridged2Bar_Pad1.0x1.5mm
- removed JP4: J_ESP_D0, Jumper:SolderJumper-2_P1.3mm_Bridged2Bar_Pad1.0x1.5mm
- removed JP5: J_ESP_3V3, Jumper:SolderJumper-2_P1.3mm_Bridged2Bar_Pad1.0x1.5mm
- removed JP6: Jumper_2_Bridged, Jumper:SolderJumper-2_P1.3mm_Bridged2Bar_Pad1.0x1.5mm
- removed KLED1 (x2), KLED10 (x2), KLED11 (x2), KLED12 (x2), KLED13 (x2), KLED14 (x2), KLED15 (x2), KLED16 (x2), KLED17 (x2), KLED18 (x2), KLED19 (x2), KLED2 (x2), KLED20 (x2), KLED21 (x2), KLED22 (x2), KLED23 (x2), KLED24 (x2), KLED25 (x2), KLED26 (x2), KLED27 (x2), KLED28 (x2), KLED29, KLED3 (x2), KLED30, KLED31, KLED32, KLED33, KLED34, KLED35, KLED36, KLED37, KLED38, KLED39, KLED4 (x2), KLED40, KLED41, KLED42, KLED43, KLED44, KLED45, KLED46, KLED47, KLED48, KLED49, KLED5 (x2), KLED50, KLED51, KLED52, KLED53, KLED54, KLED55, KLED56, KLED57, KLED58, KLED59, KLED6 (x2), KLED60, KLED61, KLED62, KLED63, KLED64, KLED7 (x2), KLED8 (x2), KLED9 (x2): LED_ARGB, chordboard-footprints:LED_D3.0mm-4
- removed MCP1, MCP2, MCP3: MCP23017_SP, Package_SO:SOIC-28W_7.5x17.9mm_P1.27mm
- removed R1, R13, R14, R15, R16, R17, R18, R6: 10K, Resistor_THT:R_Axial_DIN0204_L3.6mm_D1.6mm_P5.08mm_Horizontal
- removed R10, R11, R12, R9: R, Resistor_THT:R_Axial_DIN0207_L6.3mm_D2.5mm_P10.16mm_Horizontal
- removed R2, R3: 200, Resistor_THT:R_Axial_DIN0204_L3.6mm_D1.6mm_P5.08mm_Horizontal
- removed R4, R5, R7, R8: 4.7K, Resistor_THT:R_Axial_DIN0204_L3.6mm_D1.6mm_P5.08mm_Horizontal
- removed RE1 (x2), RE2 (x2), RE3 (x4): Rotary_Encoder, Rotary_Encoder:RotaryEncoder_Alps_EC11E_Vertical_H20mm
- removed SW1 (x2), SW10 (x2), SW11 (x2), SW12 (x2), SW13 (x2), SW14 (x2), SW15 (x2), SW16 (x2), SW17 (x2), SW18 (x2), SW19 (x2), SW2 (x2), SW20 (x2), SW21 (x2), SW22 (x2), SW23 (x2), SW24 (x2), SW25 (x2), SW26 (x2), SW27 (x2), SW28 (x2), SW29, SW3 (x2), SW30, SW31, SW32, SW33, SW34, SW35, SW36, SW37, SW38, SW39, SW4 (x2), SW40, SW41, SW42, SW43, SW44, SW45, SW46, SW47, SW48, SW5 (x2), SW6 (x2), SW7 (x2), SW8 (x2), SW9 (x2): SW_Push, chordboard-footprints:CHERRY_PCB_100H
- removed U4: MCP73832-2-OT, Package_TO_SOT_SMD:SOT-23-5
- added H7: MountingHole, MountingHole:MountingHole_2.7mm_M2.5_Pad_Via, F.Cu at (207.0, 54.6)
- added H8: MountingHole, MountingHole:MountingHole_2.7mm_M2.5_Pad_Via, F.Cu at (54.6, 54.6)
- added J10: ++5V_IN, TerminalBlock_Phoenix:TerminalBlock_Phoenix_MKDS-1,5-2_1x02_P5.00mm_Horizontal, F.Cu at (121.9, 120.7)
- added J11: T_UART4, Connector_JST:JST_PH_B4B-PH-K_1x04_P2.00mm_Vertical, F.Cu at (153.7, 123.2)
- added J12: T_I2C0_3V, Connector_JST:JST_PH_B4B-PH-K_1x04_P2.00mm_Vertical, F.Cu at (199.4, 93.3)
- added J13: T_I2C0_5V, Connector_JST:JST_PH_B4B-PH-K_1x04_P2.00mm_Vertical, F.Cu at (199.4, 123.8)
- added J14: Conn_01x08, Connector_PinHeader_2.54mm:PinHeader_1x08_P2.54mm_Vertical, F.Cu at (188.6, 88.9)
- added J15: E_UART1, Connector_JST:JST_PH_B4B-PH-K_1x04_P2.00mm_Vertical, F.Cu at (106.7, 76.8)
- added J16: T_I2C0_5V, Connector_JST:JST_PH_B4B-PH-K_1x04_P2.00mm_Vertical, F.Cu at (199.4, 117.5)
- added J8: T_UART5, Connector_JST:JST_PH_B4B-PH-K_1x04_P2.00mm_Vertical, F.Cu at (153.7, 116.8)
- added J9: Conn_01x04, Connector_PinHeader_2.54mm:PinHeader_1x04_P2.54mm_Vertical, F.Cu at (165.7, 99.1)
- added Q1: 2N7000, Package_TO_SOT_THT:TO-92_Inline, F.Cu at (205.7, 100.3)
- added Q2: 2N7000, Package_TO_SOT_THT:TO-92_Inline, F.Cu at (205.7, 106.7)
- added R27: 10K, Resistor_THT:R_Axial_DIN0204_L3.6mm_D1.6mm_P5.08mm_Horizontal, F.Cu at (64.1, 65.4)
- added R28: 200, Resistor_THT:R_Axial_DIN0204_L3.6mm_D1.6mm_P5.08mm_Horizontal, F.Cu at (64.1, 73.0)
- added R29: 200, Resistor_THT:R_Axial_DIN0204_L3.6mm_D1.6mm_P5.08mm_Horizontal, F.Cu at (203.8, 61.6)
- added R30: 4.7K, Resistor_THT:R_Axial_DIN0204_L3.6mm_D1.6mm_P5.08mm_Horizontal, F.Cu at (95.9, 66.7)
- added R31: 4.7K, Resistor_THT:R_Axial_DIN0204_L3.6mm_D1.6mm_P5.08mm_Horizontal, F.Cu at (95.9, 69.2)
- added R32: 10K, Resistor_THT:R_Axial_DIN0204_L3.6mm_D1.6mm_P5.08mm_Horizontal, F.Cu at (101.0, 75.6)
- added R35: R, Resistor_THT:R_Axial_DIN0204_L3.6mm_D1.6mm_P5.08mm_Horizontal, F.Cu at (208.9, 92.7)
- added R36: R, Resistor_THT:R_Axial_DIN0204_L3.6mm_D1.6mm_P5.08mm_Horizontal, F.Cu at (208.9, 95.2)
- added R37: R, Resistor_THT:R_Axial_DIN0204_L3.6mm_D1.6mm_P5.08mm_Horizontal, F.Cu at (208.9, 116.2)
- added R38: R, Resistor_THT:R_Axial_DIN0204_L3.6mm_D1.6mm_P5.08mm_Horizontal, F.Cu at (208.9, 113.7)
- C10: value C_Small -> 100uF; footprint Capacitor_THT:C_Disc_D3.0mm_W2.0mm_P2.50mm -> Capacitor_THT:CP_Radial_D5.0mm_P2.00mm
- C11: renamed from C5; moved to F.Cu
- C13, C14, C15, C16, DIPSW1, HLED2, RSW1, RSW2, TEE1, U1, U2: moved to F.Cu
- C7, C8: value C_Small -> C; footprint Capacitor_THT:C_Disc_D3.0mm_W2.0mm_P2.50mm -> Capacitor_THT:C_Disc_D3.0mm_W1.6mm_P2.50mm
- C9: value C_Small -> 10uF; footprint Capacitor_THT:C_Disc_D3.0mm_W2.0mm_P2.50mm -> Capacitor_THT:CP_Radial_D5.0mm_P2.00mm
- J1: value T_UART0 -> T_I2C0_3V; footprint Connector_PinHeader_2.54mm:PinHeader_1x06_P2.54mm_Vertical -> Connector_JST:JST_PH_B4B-PH-K_1x04_P2.00mm_Vertical
- J2: value E_I2C0 -> T_I2C0_5V
- J3: value E_UART0 -> Conn_01x03; footprint Connector_PinHeader_2.54mm:PinHeader_1x06_P2.54mm_Vertical -> Connector_JST:JST_EH_B03B-EH-A_1x03_P2.50mm_Vertical
- J4: value T_UART5 -> E_UART2; moved to F.Cu
- J5: value T_I2C0 -> T_UART0; footprint Connector_JST:JST_PH_B4B-PH-K_1x04_P2.00mm_Vertical -> Connector_PinHeader_2.54mm:PinHeader_1x06_P2.54mm_Vertical; moved to F.Cu
- J6: value ++5V_IN -> E_I2C0; footprint TerminalBlock_Phoenix:TerminalBlock_Phoenix_MKDS-1,5-2_1x02_P5.00mm_Horizontal -> Connector_JST:JST_PH_B4B-PH-K_1x04_P2.00mm_Vertical; moved to F.Cu
- J7: value Conn_01x07 -> E_UART0; footprint Connector_PinHeader_2.54mm:PinHeader_1x07_P2.54mm_Vertical -> Connector_PinHeader_2.54mm:PinHeader_1x06_P2.54mm_Vertical; moved to F.Cu
- JP1: value J_ESP_RX2 -> Jumper_2_Bridged
- JP10: value J_HT_AD -> J_ESP_D0; footprint Jumper:SolderJumper-2_P1.3mm_Open_Pad1.0x1.5mm -> Jumper:SolderJumper-2_P1.3mm_Bridged2Bar_Pad1.0x1.5mm; moved to B.Cu
- JP11: value J_HT_AD -> J_ESP_3V3; footprint Jumper:SolderJumper-2_P1.3mm_Open_Pad1.0x1.5mm -> Jumper:SolderJumper-2_P1.3mm_Bridged2Bar_Pad1.0x1.5mm; moved to B.Cu
- JP12: value J_HT_AD -> Jumper_2_Bridged; moved to B.Cu
- JP13: value J_HT_AD -> J_PWR_3V3; footprint Jumper:SolderJumper-2_P1.3mm_Open_Pad1.0x1.5mm -> Jumper:SolderJumper-2_P1.3mm_Bridged2Bar_Pad1.0x1.5mm; moved to B.Cu
- JP14: value J_HT_AD -> J_PWR_GND; footprint Jumper:SolderJumper-2_P1.3mm_Open_Pad1.0x1.5mm -> Jumper:SolderJumper-2_P1.3mm_Bridged2Bar_Pad1.0x1.5mm; moved to B.Cu
- JP2: value J_ESP_TX2 -> Jumper_2_Open; footprint Jumper:SolderJumper-2_P1.3mm_Bridged2Bar_Pad1.0x1.5mm -> Jumper:SolderJumper-2_P1.3mm_Open_Pad1.0x1.5mm
- JP7: value J_PWR_3V3 -> J_ESP_RX2
- JP8: value J_PWR_GND -> J_ESP_TX2
- JP9: value J_HT_AD -> J_ESP_RST; footprint Jumper:SolderJumper-2_P1.3mm_Open_Pad1.0x1.5mm -> Jumper:SolderJumper-2_P1.3mm_Bridged2Bar_Pad1.0x1.5mm; moved to B.Cu
- MEM1, MEM2, MEM3, MEM4, MEM5, MEM6: footprint Package_SO:SOIC-8_3.9x4.9mm_P1.27mm -> Package_SO:SOIJ-8_5.3x5.3mm_P1.27mm; moved to F.Cu
- U3: value 74LS126 -> DMPCM5102; footprint Package_SO:SOIC-14_3.9x8.7mm_P1.27mm -> chordboard-footprints:DMPCM5102_BLACK; moved to F.Cu
- moved MEM5 512.7 mm to (127.6, 80.6), turned to 0 degrees
- moved H3 512.0 mm to (54.6, 121.9)
- moved U3 503.2 mm to (91.4, 103.5), turned to 270 degrees
- moved MEM6 501.7 mm to (147.3, 80.6), turned to 0 degrees
- moved TEE1 496.7 mm to (177.2, 83.8)
- moved MEM3 494.3 mm to (127.6, 71.1), turned to 0 degrees
- moved MEM4 483.3 mm to (147.3, 71.1), turned to 0 degrees
- moved C7 477.4 mm to (62.2, 62.2), turned to 90 degrees
- moved MEM1 476.0 mm to (127.6, 61.6), turned to 0 degrees
- moved MEM2 465.5 mm to (147.3, 61.6), turned to 0 degrees
- moved JP14 447.0 mm to (111.1, 116.9), turned to 90 degrees
- moved J3 441.9 mm to (102.9, 123.2)
- moved C8 434.6 mm to (64.8, 62.2), turned to 90 degrees
- moved JP12 429.2 mm to (111.8, 57.8), turned to 180 degrees
- moved JP11 426.4 mm to (111.8, 60.3), turned to 180 degrees
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Connections:
- C10 pad 2: /T_GND -> GND
- C11 pad 1: +3V3 -> /T_3V3
- C12 pad 1: /RE1B -> /T_3V3
- C13 pad 1: /RE2A -> /T_3V3
- C14 pad 1: /RE2B -> /T_3V3
- C15 pad 1: /RE3A -> /T_3V3
- C16 pad 1: /RE3B -> /T_3V3
- C7 pad 1: +3V3 -> /ESP_3V3
- C7 pad 2: /T_GND -> /ESP_GND
- C8 pad 1: +3V3 -> /ESP_3V3
- C8 pad 2: /T_GND -> /ESP_GND
- C9 pad 1: +3V3 -> +5V
- C9 pad 2: /T_GND -> GND
- D3 pad 1: Net-(D3-Pad1) -> +5V
- D3 pad 2: /COM_AD2 -> Net-(D3-Pad2)
- J1 pad 1: /T_GND -> /T_SCL
- J1 pad 2: (no net) -> /T_SDA
- J1 pad 3: (no net) -> /T_3V3
- J1 pad 4: /T_RX1 -> /T_GND
- J2 pad 1: /ESP_SCL -> /T_SCL5
- J2 pad 2: /ESP_SDA -> /T_SDA5
- J2 pad 3: /ESP_3V3 -> +5V
- J2 pad 4: /ESP_GND -> /T_GND
- J3 pad 1: /ESP_GND -> Net-(J3-Pad1)
- J3 pad 2: (no net) -> Net-(J3-Pad2)
- J3 pad 3: (no net) -> Net-(J3-Pad3)
- J4 pad 1: Net-(J4-Pad1) -> /T_RX4
- J4 pad 2: Net-(J4-Pad2) -> /T_TX4
- J4 pad 3: +3V3 -> (no net)
- J4 pad 4: /T_GND -> /ESP_GND
- J5 pad 1: /T_SCL -> /T_GND
- J5 pad 2: /T_SDA -> (no net)
- J5 pad 3: +3V3 -> (no net)
- J5 pad 4: /T_GND -> /T_RX1
- J6 pad 1: Net-(D1-Pad2) -> /ESP_SCL
- J6 pad 2: GND -> /ESP_SDA
- J7 pad 1: /MEMCARD_CS1 -> /ESP_GND
- J7 pad 2: /MEMCARD_CS2 -> (no net)
- J7 pad 3: /MEMCARD_CS3 -> (no net)
- J7 pad 4: /MEMCARD_CS4 -> /ESP_RX0
- J7 pad 5: /MEMCARD_MOSI -> /ESP_TX0
- J7 pad 6: /MEMCARD_MISO -> (no net)
- JP1 pad 1: /T_TX4 -> /DAC_GND
- JP1 pad 2: /ESP_RX2 -> /T_GND
- JP10 pad 2: Net-(HT2-Pad24) -> /ESP_D0
- JP11 pad 1: Net-(JP11-Pad1) -> /T_3V3
- JP11 pad 2: Net-(HT2-Pad25) -> /ESP_3V3
- JP12 pad 1: Net-(JP12-Pad1) -> /T_GND
- JP12 pad 2: Net-(HT1-Pad23) -> /ESP_GND
- JP13 pad 1: Net-(JP13-Pad1) -> +3V3
- JP13 pad 2: Net-(HT1-Pad24) -> /T_3V3
- JP14 pad 1: Net-(JP14-Pad1) -> GND
- JP14 pad 2: Net-(HT1-Pad25) -> /T_GND
- JP2 pad 1: /T_RX4 -> /DAC_3V3
- JP2 pad 2: /ESP_TX2 -> +5V
- JP7 pad 1: +3V3 -> /T_TX4
- JP7 pad 2: +3V3 -> /ESP_RX2
- JP8 pad 1: GND -> /T_RX4
- JP8 pad 2: /T_GND -> /ESP_TX2
- JP9 pad 2: Net-(HT2-Pad23) -> /ESP_RST
- MEM1 pad 3: +3V3 -> /T_3V3
- MEM1 pad 7: +3V3 -> /T_3V3
- MEM1 pad 8: +3V3 -> /T_3V3
- MEM2 pad 3: +3V3 -> /T_3V3
- MEM2 pad 7: +3V3 -> /T_3V3
- MEM2 pad 8: +3V3 -> /T_3V3
- MEM3 pad 3: +3V3 -> /T_3V3
- MEM3 pad 7: +3V3 -> /T_3V3
- MEM3 pad 8: +3V3 -> /T_3V3
- MEM4 pad 3: +3V3 -> /T_3V3
- MEM4 pad 7: +3V3 -> /T_3V3
- MEM4 pad 8: +3V3 -> /T_3V3
- MEM5 pad 1: /MEMCARD_CS4 -> /MEMCARD_CS5
- MEM5 pad 3: +3V3 -> /T_3V3
- MEM5 pad 7: +3V3 -> /T_3V3
- MEM5 pad 8: +3V3 -> /T_3V3
- MEM6 pad 1: /MEMCARD_CS4 -> /MEMCARD_CS6
- MEM6 pad 3: +3V3 -> /T_3V3
- MEM6 pad 7: +3V3 -> /T_3V3
- MEM6 pad 8: +3V3 -> /T_3V3
- TEE1 pad 10: (no net) -> /MEMCARD_CS6
- TEE1 pad 15: +3V3 -> /T_3V3
- TEE1 pad 17: Net-(JP3-Pad1) -> Net-(JP9-Pad1)
- TEE1 pad 18: Net-(JP4-Pad1) -> Net-(JP10-Pad1)
- TEE1 pad 19: (no net) -> Net-(J9-Pad1)
- TEE1 pad 20: (no net) -> Net-(J9-Pad2)
- TEE1 pad 21: (no net) -> Net-(J9-Pad3)
- TEE1 pad 22: (no net) -> Net-(J9-Pad4)
- TEE1 pad 25: Net-(J4-Pad2) -> /TX5
- TEE1 pad 26: Net-(J4-Pad1) -> /RX5
- TEE1 pad 27: /RE2B -> Net-(J14-Pad8)
- TEE1 pad 28: /RE2A -> Net-(J14-Pad7)
- TEE1 pad 29: /RE1B -> Net-(J14-Pad6)
- TEE1 pad 30: /RE1A -> Net-(J14-Pad5)
- TEE1 pad 31: (no net) -> Net-(J14-Pad4)
- TEE1 pad 32: (no net) -> Net-(J14-Pad3)
- TEE1 pad 33: (no net) -> Net-(J14-Pad2)
- TEE1 pad 34: (no net) -> Net-(J14-Pad1)
- TEE1 pad 38: /RE3B -> (no net)
- TEE1 pad 39: /RE3A -> (no net)
- TEE1 pad 48: /T_5V -> +5V
- TEE1 pad 8: (no net) -> /MEMCARD_CS5
- U1 pad 10: (no net) -> Net-(U1-Pad10)
- U1 pad 11: (no net) -> Net-(U1-Pad11)
- U1 pad 12: (no net) -> Net-(U1-Pad12)
- U3 pad 1: (no net) -> +5V
- U3 pad 10: (no net) -> /DAC_GND
- U3 pad 11: (no net) -> /DAC_3V3
- U3 pad 12: (no net) -> Net-(J3-Pad1)
- U3 pad 13: (no net) -> Net-(J3-Pad2)
- U3 pad 14: (no net) -> Net-(J3-Pad3)
- U3 pad 2: (no net) -> /DAC_3V3
- U3 pad 3: (no net) -> /DAC_GND
- U3 pad 4: (no net) -> /DAC_GND
- U3 pad 5: (no net) -> /DAC_GND
- U3 pad 6: (no net) -> /DAC_GND
- U3 pad 7: (no net) -> Net-(U1-Pad12)
- U3 pad 8: (no net) -> Net-(U1-Pad11)
- U3 pad 9: (no net) -> Net-(U1-Pad10)
Routing:
- net /T_GND: track 0.00 -> 390.9 mm, vias 0 -> 3
- net /T_3V3: track 0.00 -> 338.8 mm, vias 0 -> 2
- net +5V: track 0.00 -> 229.4 mm
- net /T_RX4: track 0.00 -> 157.3 mm
- net /ESP_GND: track 0.00 -> 156.9 mm, vias 0 -> 2
- net /T_TX4: track 0.00 -> 153.9 mm
- net /MEMCARD_SCK: track 0.00 -> 149.1 mm, vias 0 -> 3
- net /ESP_RST: track 0.00 -> 126.9 mm, vias 0 -> 2
- net /MEMCARD_MISO: track 0.00 -> 114.3 mm, vias 0 -> 4
- net /ESP_RX2: track 0.00 -> 107.6 mm, vias 0 -> 1
- net /MEMCARD_MOSI: track 0.00 -> 104.2 mm, vias 0 -> 3
- net /ESP_TX2: track 0.00 -> 102.4 mm, vias 0 -> 1
- net /ESP_D0: track 0.00 -> 94.2 mm, vias 0 -> 1
- net /ESP_3V3: track 0.00 -> 80.5 mm, vias 0 -> 2
- net /T_RX1: track 0.00 -> 64.0 mm
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Other:
- board size 302.9 x 193 mm -> 161.3 x 76.2 mm
- net class Default: trace_width 0.4 -> 0.7
