File: hard/v2.0/chordboard/chordboard.sch (KiCad schematic (older format))
At the start: 136 parts, among them J1 T_I2C0, J10 ++5V_IN, J11 Conn_01x07, J12 T_I2C0, J13 T_I2C0, J2 T_I2C0, J3 Conn_02x20_Odd_Even, J4 Conn_02x20_Odd_Even, J5 T_UART0, J6 E_I2C0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

Commit message: Updated
Parts:
- removed C1, C2: C_Small, Capacitor_THT:C_Disc_D3.4mm_W2.1mm_P2.50mm, symbol Device:C_Small
- removed C17, C18: C_Small, Capacitor_SMD:C_0603_1608Metric_Pad1.05x0.95mm_HandSolder, symbol Device:C_Small
- removed C19: C_Small, Capacitor_THT:C_Disc_D3.0mm_W2.0mm_P2.50mm, symbol Device:C_Small
- removed C3, C4, C5, C6: C, Capacitor_THT:C_Disc_D3.4mm_W2.1mm_P2.50mm, symbol Device:C
- removed D1, D2: D, Diode_THT:D_DO-41_SOD81_P7.62mm_Horizontal, symbol Device:D
- removed H1, H10, H11, H12, H13, H14, H2, H5, H6, H9: MountingHole, MountingHole:MountingHole_2.7mm_M2.5_Pad_Via, symbol Mechanical:MountingHole
- removed HT1, HT2: HT16K33, Package_SO:SOIC-28W_7.5x17.9mm_P1.27mm, symbol eurocad:HT16K33
- removed IO1, IO2: MCP23017_SO, Package_SO:SOIC-28W_7.5x17.9mm_P1.27mm, symbol Interface_Expansion:MCP23017_SO
- removed J11: Conn_01x07, Connector_PinHeader_2.54mm:PinHeader_1x07_P2.54mm_Vertical, symbol Connector_Generic:Conn_01x07
- removed J3, J4: Conn_02x20_Odd_Even, Connector_IDC:IDC-Header_2x20_P2.54mm_Vertical, symbol Connector_Generic:Conn_02x20_Odd_Even
- removed J9: T_I2C0, Connector_JST:JST_PH_B4B-PH-K_1x04_P2.00mm_Vertical, symbol chordboard-components:GROVE_I2C
- removed JP2, JP3, JP4, JP5, JP6: J_HT_AD, Jumper:SolderJumper-2_P1.3mm_Open_Pad1.0x1.5mm, symbol Jumper:Jumper_2_Bridged
- removed MCP1: MCP23017_SP, Package_SO:SOIC-28W_7.5x17.9mm_P1.27mm, symbol Interface_Expansion:MCP23017_SP
- removed Q1, Q2: BSS138, TO_SOT_Packages_SMD:SOT-23, symbol chordboard-rescue:BSS138-Transistor-leftpad-rescue
- removed R1, R2, R3, R4, R5, R6: 10K, Resistor_THT:R_Axial_DIN0204_L3.6mm_D1.6mm_P5.08mm_Horizontal, symbol Device:R
- removed R10, R11, R12, R13, R14, R15, R16, R17, R18, R19, R20, R21, R22, R23, R24, R25, R26, R7, R8, R9: 39K, Resistor_THT:R_Axial_DIN0204_L3.6mm_D1.6mm_P5.08mm_Horizontal, symbol Device:R
- removed R33, R34: 4.7K, Resistor_THT:R_Axial_DIN0204_L3.6mm_D1.6mm_P5.08mm_Horizontal, symbol chordboard-components:R
- removed RE1, RE10, RE11, RE12, RE2, RE3, RE4, RE5, RE6, RE7, RE8, RE9: Rotary_Encoder, Rotary_Encoder:RotaryEncoder_Alps_EC11E_Vertical_H20mm, symbol Device:Rotary_Encoder
- removed U3: 74LS126, Package_SO:SOIC-14_3.9x8.7mm_P1.27mm, symbol 74xx:74LS126
- removed U4: MCP73832-2-OT, Package_TO_SOT_SMD:SOT-23-5, symbol Battery_Management:MCP73832-2-OT
- added J11: T_UART4, Connector_JST:JST_PH_B4B-PH-K_1x04_P2.00mm_Vertical, symbol chordboard-components:GROVE_UART
- added J14: Conn_01x08, Connector_PinHeader_2.54mm:PinHeader_1x08_P2.54mm_Vertical, symbol Connector_Generic:Conn_01x08
- added J15: E_UART1, Connector_JST:JST_PH_B4B-PH-K_1x04_P2.00mm_Vertical, symbol chordboard-components:GROVE_UART
- added J16: T_I2C0_5V, Connector_JST:JST_PH_B4B-PH-K_1x04_P2.00mm_Vertical, symbol chordboard-components:GROVE_I2C
- added J3: Conn_01x03, Connector_JST:JST_EH_B03B-EH-A_1x03_P2.50mm_Vertical, symbol Connector_Generic:Conn_01x03
- added J4: E_UART2, Connector_JST:JST_PH_B4B-PH-K_1x04_P2.00mm_Vertical, symbol chordboard-components:GROVE_UART
- added J9: Conn_01x04, Connector_PinHeader_2.54mm:PinHeader_1x04_P2.54mm_Vertical, symbol Connector_Generic:Conn_01x04
- added JP2: Jumper_2_Open, Jumper:SolderJumper-2_P1.3mm_Open_Pad1.0x1.5mm, symbol Jumper:Jumper_2_Open
- added Q1, Q2: 2N7000, Package_TO_SOT_THT:TO-92_Inline, symbol Transistor_FET:2N7000
- added U3: DMPCM5102, chordboard-footprints:DMPCM5102_BLACK, symbol chordboard-components:DMPCM5102
- J1, J12: value T_I2C0 -> T_I2C0_3V
- J13, J2: value T_I2C0 -> T_I2C0_5V
- JP1: value J_HT_AD -> Jumper_2_Bridged; footprint Jumper:SolderJumper-2_P1.3mm_Open_Pad1.0x1.5mm -> Jumper:SolderJumper-2_P1.3mm_Bridged2Bar_Pad1.0x1.5mm
- MEM1, MEM2, MEM3, MEM4, MEM5, MEM6: footprint Package_SO:SOIC-8_3.9x4.9mm_P1.27mm -> Package_SO:SOIJ-8_5.3x5.3mm_P1.27mm
- R35, R36, R37, R38: footprint Resistor_THT:R_Axial_DIN0207_L6.3mm_D2.5mm_P10.16mm_Horizontal -> Resistor_THT:R_Axial_DIN0204_L3.6mm_D1.6mm_P5.08mm_Horizontal
Connections:
- net labels added: DAC_3V3, DAC_GND, ESP_3V, RX5, TX5
- net labels removed: E_ROTARY_INTA, E_ROTARY_INTB, LED_CLK, LED_CS, LED_DAT, RE1A, RE1B, RE2A, RE2B, SCL5, SDA5
- wire segments 462 -> 153
Other:
- moved on the sheet: C11, C12, C13, C14, C15, C16, H3, H4, J1, J12, J13, J2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
