File: hard/v2.0/controlpad/chordboard.kicad_pcb (KiCad board)
At the start: 2 copper layers, 152.4 x 76.2 mm, 89 parts, among them J1 Conn_02x20_Odd_Even, SW1 SW_Push, SW10 SW_Push, SW11 SW_Push, SW12 SW_Push, SW13 SW_Push, SW14 SW_Push, SW15 SW_Push, SW16 SW_Push, SW17 SW_Push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

Commit message: Updated
Parts:
- added J2: GROVE_I2C, Connector_JST:JST_PH_B4B-PH-K_1x04_P2.00mm_Vertical, B.Cu at (247.0, 149.9)
Connections:
- J1 pad 34: (no net) -> /T_SCL
- J1 pad 36: (no net) -> /T_SDA
- J1 pad 38: (no net) -> /T_5V
- J1 pad 40: (no net) -> /T_GND
Routing:
- net Net-(J1-Pad37): track 0.00 -> 396.9 mm
- net Net-(J1-Pad35): track 0.00 -> 374.8 mm
- net Net-(J1-Pad31): track 0.00 -> 341.2 mm
- net Net-(J1-Pad39): track 0.00 -> 324.5 mm
- net Net-(J1-Pad29): track 0.00 -> 313.9 mm
- net Net-(J1-Pad33): track 0.00 -> 267.5 mm, vias 0 -> 1
- net /KR7: track 0.00 -> 237.2 mm, vias 0 -> 2
- net /KR2: track 0.00 -> 220.4 mm, vias 0 -> 2
- net /KS0: track 0.00 -> 205.9 mm
- net /KR3: track 0.00 -> 205.7 mm
- net Net-(J1-Pad27): track 0.00 -> 204.2 mm
- net Net-(J1-Pad23): track 0.00 -> 196.6 mm, vias 0 -> 1
- net Net-(J1-Pad25): track 0.00 -> 192.4 mm
- net /KR8: track 0.00 -> 186.0 mm, vias 0 -> 1
- net /KR9: track 0.00 -> 169.9 mm
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Other:
- outline, holes or cut-outs redrawn
