File: hard/v2.0/controlpad/chordboard.sch (KiCad schematic (older format))
At the start: 89 parts, among them J4 Conn_02x20_Odd_Even, SW1 SW_Push, SW10 SW_Push, SW11 SW_Push, SW12 SW_Push, SW13 SW_Push, SW14 SW_Push, SW15 SW_Push, SW16 SW_Push, SW17 SW_Push, SW18 SW_Push, SW19 SW_Push, SW2 SW_Push, SW20 SW_Push, SW21 SW_Push, SW22 SW_Push, SW23 SW_Push, SW24 SW_Push, SW25 SW_Push, SW26 SW_Push, SW27 SW_Push, SW28 SW_Push, SW3 SW_Push, SW4 SW_Push, SW5 SW_Push, SW6 SW_Push, SW7 SW_Push, SW8 SW_Push, SW9 SW_Push

Commit message: Updated
Parts:
- added J2: GROVE_I2C, Connector_JST:JST_PH_B4B-PH-K_1x04_P2.00mm_Vertical, symbol chordboard-components:GROVE_I2C
- renumbered D4 to D1, D3 to D10, D6 to D11, D9 to D12, D12 to D13, D15 to D14, D18 to D15, D21 to D16, D24 to D17, D27 to D18, D2 to D19, D7 to D2, D5 to D20, D8 to D21, D11 to D22, D14 to D23, D17 to D24, D20 to D25, D23 to D26, D26 to D27, D29 to D28, D10 to D3, D13 to D4, D16 to D5, D19 to D6, D22 to D7, D25 to D8, D28 to D9, J4 to J1, KLED17 to KLED15, KLED18 to KLED16, KLED19 to KLED17, KLED20 to KLED18, KLED21 to KLED19, KLED22 to KLED20, KLED23 to KLED21, KLED24 to KLED22, KLED25 to KLED23, KLED26 to KLED24, KLED27 to KLED25, KLED28 to KLED26, KLED29 to KLED27, KLED30 to KLED28, SW3 to SW1, SW2 to SW10, SW5 to SW11, SW8 to SW12, SW11 to SW13, SW17 to SW15, SW20 to SW16, SW23 to SW17, SW26 to SW18, SW1 to SW19, SW6 to SW2, SW4 to SW20, SW7 to SW21, SW10 to SW22, SW13 to SW23, SW16 to SW24, SW19 to SW25, SW22 to SW26, SW25 to SW27, SW9 to SW3, SW12 to SW4, SW15 to SW5, SW18 to SW6, SW21 to SW7, SW24 to SW8, SW27 to SW9
Connections:
- net labels added: T_5V, T_GND, T_SCL, T_SDA
- wire segments 501 -> 505
Other:
- moved on the sheet: H1, H2, H3, H4
